Commit message: Add ros2_control to urdf, update relevant config to match kuka_experimental

File: src/cybertech_mock/description/kuka_cybertech.urdf.xacro (robot description, xacro)
@@ -1,19 +1,6 @@
-<?xml version="1.0" ?>
+<?xml version="1.0"?>
 <robot name="kuka_cybertech" xmlns:xacro="http://wiki.ros.org/xacro">
-  <!-- <xacro:arg name="robot_model" default="$(arg robot_model)"/>
-  <xacro:arg name="robot_ip" default="$(arg robot_ip)"/>
-  <xacro:arg name="rmi_port" default="16001"/>
-  <xacro:arg name="stream_motion_port" default="60015"/>
-  <xacro:arg name="gpio_configuration" default="$(find fanuc_hardware_interface)/config/example_gpio_config.yaml"/>
-  <xacro:arg name="payload_schedule" default="1"/>
-  <xacro:arg name="use_mock" default="false"/> -->
-  <xacro:include filename="$(find kuka_kr16_support)/urdf/kr16_2_macro.xacro" />
-  <!-- <xacro:if value="$(arg use_mock)">
-    <xacro:include filename="$(find fanuc_hardware_interface)/config/cybertech_mock_ros2_control_macro.xacro"/>
-  </xacro:if>
-  <xacro:unless value="$(arg use_mock)">
-    <xacro:include filename="$(find fanuc_hardware_interface)/config/crx_physical_ros2_control_macro.xacro"/>
-  </xacro:unless> -->
-  <link name="world"/>
+  <xacro:include filename="$(find kuka_ros2_control_support)/urdf/common_kuka.xacro" />
+  <link name="world" />
   <joint name="world-base_link" type="fixed">
     <origin xyz="0 0 0" rpy="0 0 0" />
@@ -21,5 +8,5 @@
     <child link="base_link" />
   </joint>
-  <link name="grasp_link"/>
+  <link name="grasp_link" />
   <joint name="flange-grasp_link" type="fixed">
     <origin xyz="0 0 0" rpy="${radians(90)} 0 ${radians(90)}" />
@@ -27,5 +14,3 @@
     <child link="grasp_link" />
   </joint>
-  <xacro:kuka_kr16_2 prefix=""/>
-  <!-- <xacro:crx_control name="$(arg robot_model)"/> -->
 </robot>
